Commit message: Use xacro builtin pi constant

File: velodyne_description/urdf/HDL-32E.urdf.xacro (robot description, xacro)
@@ -1,6 +1,5 @@
 <?xml version="1.0"?>
 <robot xmlns:xacro="http://www.ros.org/wiki/xacro" name="HDL-32E">
-  <xacro:property name="M_PI" value="3.1415926535897931" />
-  <xacro:macro name="HDL-32E" params="*origin parent:=base_link name:=velodyne topic:=/velodyne_points hz:=10 lasers:=32 samples:=2187 collision_range:=0.3 min_range:=0.9 max_range:=130.0 noise:=0.008 min_angle:=-${M_PI} max_angle:=${M_PI} gpu:=false">
+  <xacro:macro name="HDL-32E" params="*origin parent:=base_link name:=velodyne topic:=/velodyne_points hz:=10 lasers:=32 samples:=2187 collision_range:=0.3 min_range:=0.9 max_range:=130.0 noise:=0.008 min_angle:=-${pi} max_angle:=${pi} gpu:=false">
     <joint name="${name}_base_mount_joint" type="fixed">
       <xacro:insert_block name="origin" />
@@ -64,6 +63,6 @@
                 <samples>${lasers}</samples>
                 <resolution>1</resolution>
-                <min_angle>-${30.67*M_PI/180.0}</min_angle>
-                <max_angle> ${10.67*M_PI/180.0}</max_angle>
+                <min_angle>-${30.67*pi/180.0}</min_angle>
+                <max_angle> ${10.67*pi/180.0}</max_angle>
               </vertical>
             </scan>
@@ -104,6 +103,6 @@
                 <samples>${lasers}</samples>
                 <resolution>1</resolution>
-                <min_angle>-${30.67*M_PI/180.0}</min_angle>
-                <max_angle> ${10.67*M_PI/180.0}</max_angle>
+                <min_angle>-${30.67*pi/180.0}</min_angle>
+                <max_angle> ${10.67*pi/180.0}</max_angle>
               </vertical>
             </scan>

File: velodyne_description/urdf/VLP-16.urdf.xacro (robot description, xacro)
@@ -1,6 +1,5 @@
 <?xml version="1.0"?>
 <robot xmlns:xacro="http://www.ros.org/wiki/xacro" name="VLP-16">
-  <xacro:property name="M_PI" value="3.1415926535897931"/>
-  <xacro:macro name="VLP-16" params="*origin parent:=base_link name:=velodyne topic:=/velodyne_points hz:=10 lasers:=16 samples:=1875 collision_range:=0.3 min_range:=0.9 max_range:=130.0 noise:=0.008 min_angle:=-${M_PI} max_angle:=${M_PI} gpu:=false">
+  <xacro:macro name="VLP-16" params="*origin parent:=base_link name:=velodyne topic:=/velodyne_points hz:=10 lasers:=16 samples:=1875 collision_range:=0.3 min_range:=0.9 max_range:=130.0 noise:=0.008 min_angle:=-${pi} max_angle:=${pi} gpu:=false">
     <joint name="${name}_base_mount_joint" type="fixed">
       <xacro:insert_block name="origin"/>
@@ -67,7 +66,6 @@
                 <samples>${lasers}</samples>
                 <resolution>1</resolution>
-                <min_angle>-${15.0*M_PI/180.0}</min_angle>
-                <max_angle>
-                  ${15.0*M_PI/180.0}</max_angle>
+                <min_angle>-${15.0*pi/180.0}</min_angle>
+                <max_angle> ${15.0*pi/180.0}</max_angle>
               </vertical>
             </scan>
@@ -108,7 +106,6 @@
                 <samples>${lasers}</samples>
                 <resolution>1</resolution>
-                <min_angle>-${15.0*M_PI/180.0}</min_angle>
-                <max_angle>
-                  ${15.0*M_PI/180.0}</max_angle>
+                <min_angle>-${15.0*pi/180.0}</min_angle>
+                <max_angle> ${15.0*pi/180.0}</max_angle>
               </vertical>
             </scan>

File: velodyne_description/urdf/VLP-32C.urdf.xacro (robot description, xacro)
@@ -1,6 +1,5 @@
 <?xml version="1.0"?>
 <robot xmlns:xacro="http://www.ros.org/wiki/xacro" name="VLP-32C">
-  <xacro:property name="M_PI" value="3.1415926535897931"/>
-  <xacro:macro name="VLP-32C" params="*origin parent:=base_link name:=velodyne topic:=/velodyne_points hz:=10 lasers:=32 samples:=1200 collision_range:=0.3 min_range:=0.4 max_range:=200.0 noise:=0.008 min_angle:=-${M_PI} max_angle:=${M_PI} gpu:=false">
+  <xacro:macro name="VLP-32C" params="*origin parent:=base_link name:=velodyne topic:=/velodyne_points hz:=10 lasers:=32 samples:=1200 collision_range:=0.3 min_range:=0.4 max_range:=200.0 noise:=0.008 min_angle:=-${pi} max_angle:=${pi} gpu:=false">
     <joint name="${name}_base_mount_joint" type="fixed">
       <xacro:insert_block name="origin"/>
@@ -68,6 +67,6 @@
                 <samples>${2 * lasers}</samples>
                 <resolution>1</resolution>
-                <min_angle>${-25.0*M_PI/180.0}</min_angle>
-                <max_angle>${15.0*M_PI/180.0}</max_angle>
+                <min_angle>${-25.0*pi/180.0}</min_angle>
+                <max_angle>${15.0*pi/180.0}</max_angle>
               </vertical>
             </scan>
@@ -89,12 +88,12 @@
               <vertical>
                 <angles>
-                  ${-25.000 * M_PI / 180.0}  ${-15.639 * M_PI / 180.0}  ${-11.310 * M_PI / 180.0}  ${-8.843 * M_PI / 180.0}
-                  ${ -7.254 * M_PI / 180.0}  ${ -6.148 * M_PI / 180.0}  ${ -5.333 * M_PI / 180.0}  ${-4.667 * M_PI / 180.0}
-                  ${ -4.000 * M_PI / 180.0}  ${ -3.667 * M_PI / 180.0}  ${ -3.333 * M_PI / 180.0}  ${-3.000 * M_PI / 180.0}
-                  ${ -2.667 * M_PI / 180.0}  ${ -2.333 * M_PI / 180.0}  ${ -2.000 * M_PI / 180.0}  ${-1.667 * M_PI / 180.0}
-                  ${ -1.333 * M_PI / 180.0}  ${ -1.000 * M_PI / 180.0}  ${ -0.667 * M_PI / 180.0}  ${-0.333 * M_PI / 180.0}
-                  ${  0.000 * M_PI / 180.0}  ${  0.333 * M_PI / 180.0}  ${  0.667 * M_PI / 180.0}  ${ 1.000 * M_PI / 180.0}
-                  ${  1.333 * M_PI / 180.0}  ${  1.667 * M_PI / 180.0}  ${  2.333 * M_PI / 180.0}  ${ 3.333 * M_PI / 180.0}
-                  ${  4.667 * M_PI / 180.0}  ${  7.000 * M_PI / 180.0}  ${ 10.333 * M_PI / 180.0}  ${15.000 * M_PI / 180.0}
+                  ${-25.000 * pi / 180.0}  ${-15.639 * pi / 180.0}  ${-11.310 * pi / 180.0}  ${-8.843 * pi / 180.0}
+                  ${ -7.254 * pi / 180.0}  ${ -6.148 * pi / 180.0}  ${ -5.333 * pi / 180.0}  ${-4.667 * pi / 180.0}
+                  ${ -4.000 * pi / 180.0}  ${ -3.667 * pi / 180.0}  ${ -3.333 * pi / 180.0}  ${-3.000 * pi / 180.0}
+                  ${ -2.667 * pi / 180.0}  ${ -2.333 * pi / 180.0}  ${ -2.000 * pi / 180.0}  ${-1.667 * pi / 180.0}
+                  ${ -1.333 * pi / 180.0}  ${ -1.000 * pi / 180.0}  ${ -0.667 * pi / 180.0}  ${-0.333 * pi / 180.0}
+                  ${  0.000 * pi / 180.0}  ${  0.333 * pi / 180.0}  ${  0.667 * pi / 180.0}  ${ 1.000 * pi / 180.0}
+                  ${  1.333 * pi / 180.0}  ${  1.667 * pi / 180.0}  ${  2.333 * pi / 180.0}  ${ 3.333 * pi / 180.0}
+                  ${  4.667 * pi / 180.0}  ${  7.000 * pi / 180.0}  ${ 10.333 * pi / 180.0}  ${15.000 * pi / 180.0}
                 </angles>
               </vertical>
@@ -122,6 +121,6 @@
                 <samples>${lasers}</samples>
                 <resolution>1</resolution>
-                <min_angle>${-25.0*M_PI/180.0}</min_angle>
-                <max_angle>${15.0*M_PI/180.0}</max_angle>
+                <min_angle>${-25.0*pi/180.0}</min_angle>
+                <max_angle>${15.0*pi/180.0}</max_angle>
               </vertical>
             </scan>
@@ -143,12 +142,12 @@
               <vertical>
                 <angles>
-                  ${-25.000 * M_PI / 180.0}  ${-15.639 * M_PI / 180.0}  ${-11.310 * M_PI / 180.0}  ${-8.843 * M_PI / 180.0}
-                  ${ -7.254 * M_PI / 180.0}  ${ -6.148 * M_PI / 180.0}  ${ -5.333 * M_PI / 180.0}  ${-4.667 * M_PI / 180.0}
-                  ${ -4.000 * M_PI / 180.0}  ${ -3.667 * M_PI / 180.0}  ${ -3.333 * M_PI / 180.0}  ${-3.000 * M_PI / 180.0}
-                  ${ -2.667 * M_PI / 180.0}  ${ -2.333 * M_PI / 180.0}  ${ -2.000 * M_PI / 180.0}  ${-1.667 * M_PI / 180.0}
-                  ${ -1.333 * M_PI / 180.0}  ${ -1.000 * M_PI / 180.0}  ${ -0.667 * M_PI / 180.0}  ${-0.333 * M_PI / 180.0}
-                  ${  0.000 * M_PI / 180.0}  ${  0.333 * M_PI / 180.0}  ${  0.667 * M_PI / 180.0}  ${ 1.000 * M_PI / 180.0}
-                  ${  1.333 * M_PI / 180.0}  ${  1.667 * M_PI / 180.0}  ${  2.333 * M_PI / 180.0}  ${ 3.333 * M_PI / 180.0}
-                  ${  4.667 * M_PI / 180.0}  ${  7.000 * M_PI / 180.0}  ${ 10.333 * M_PI / 180.0}  ${15.000 * M_PI / 180.0}
+                  ${-25.000 * pi / 180.0}  ${-15.639 * pi / 180.0}  ${-11.310 * pi / 180.0}  ${-8.843 * pi / 180.0}
+                  ${ -7.254 * pi / 180.0}  ${ -6.148 * pi / 180.0}  ${ -5.333 * pi / 180.0}  ${-4.667 * pi / 180.0}
+                  ${ -4.000 * pi / 180.0}  ${ -3.667 * pi / 180.0}  ${ -3.333 * pi / 180.0}  ${-3.000 * pi / 180.0}
+                  ${ -2.667 * pi / 180.0}  ${ -2.333 * pi / 180.0}  ${ -2.000 * pi / 180.0}  ${-1.667 * pi / 180.0}
+                  ${ -1.333 * pi / 180.0}  ${ -1.000 * pi / 180.0}  ${ -0.667 * pi / 180.0}  ${-0.333 * pi / 180.0}
+                  ${  0.000 * pi / 180.0}  ${  0.333 * pi / 180.0}  ${  0.667 * pi / 180.0}  ${ 1.000 * pi / 180.0}
+                  ${  1.333 * pi / 180.0}  ${  1.667 * pi / 180.0}  ${  2.333 * pi / 180.0}  ${ 3.333 * pi / 180.0}
+                  ${  4.667 * pi / 180.0}  ${  7.000 * pi / 180.0}  ${ 10.333 * pi / 180.0}  ${15.000 * pi / 180.0}
                 </angles>
               </vertical>
